File: Tesis MIB/Proyecto de Tesis/TESIS - Desarrollo/PCB/Puente H p Fuente AT/Puente_H/Puente_H.kicad_sch (KiCad schematic)
At the start: 59 parts

Commit message: actualiza info de Tesis
Incorpora archivos de simulación de propuesta de fuente en Proteus y los archivos de Kicad del mismo circuito.
Parts:
- added J2: Screw_Terminal_01x02, TerminalBlock_4Ucon:TerminalBlock_4Ucon_1x02_P3.50mm_Vertical, symbol Connector:Screw_Terminal_01x02
- C1, C4, C7, C8: renamed from C?; footprint (none) -> Capacitor_THT:C_Disc_D5.0mm_W2.5mm_P2.50mm
- C2, C3: renamed from C?; footprint (none) -> Capacitor_THT:CP_Radial_D10.0mm_P5.00mm
- C5, C6: renamed from C?; footprint (none) -> Capacitor_THT:CP_Radial_D6.3mm_P2.50mm
- D11, D12, D5, D6: renamed from D?; footprint Diode_THT:D_DO-201_P15.24mm_Horizontal -> Diode_THT:D_DO-35_SOD27_P7.62mm_Horizontal
- J1: renamed from J?; footprint (none) -> TerminalBlock_4Ucon:TerminalBlock_4Ucon_1x03_P3.50mm_Horizontal
- J3: renamed from J?; footprint (none) -> TerminalBlock_4Ucon:TerminalBlock_4Ucon_1x02_P3.50mm_Vertical
- R1, R10, R11, R12, R13, R14, R15, R16, R17, R18, R19, R2, R20, R3, R4, R5, R6, R7, R8, R9: renamed from R?; footprint (none) -> Resistor_THT:R_Axial_DIN0207_L6.3mm_D2.5mm_P7.62mm_Horizontal
- T1: renamed from T?; footprint (none) -> Transformer_THT:Transformer_NF_ETAL_1-1_P1200
- gave numbers to parts that had none: 24
Connections:
- net +5V: now also J2.1 (Pin_1)
- net GND: now also J2.2 (Pin_2)
- net at D10.1 (K), D9.2 (A), Q6.3 (S)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: now also D11.2 (A); no longer D11.1 (K)
- net at Q6.1 (G), R13.2, U6.4: now also D11.1 (K); no longer D11.2 (A)
- no-connect marks 25 -> 29
Other:
- moved on the sheet: D11, D6, J3, R12
