File: Tesis MIB/Proyecto de Tesis/TESIS - Desarrollo/PCB/Puente H p Fuente AT/Puente_H/_autosave-Puente_H.kicad_sch (KiCad schematic)
At the start: 60 parts, among them J1 Screw_Terminal_01x03, J2 Screw_Terminal_01x02, J3 Screw_Terminal_01x02, Q1 BC547, Q2 BC547, Q3 BC337, Q4 IRF3205, Q5 IRF3205, Q6 IRF3205, Q7 IRF3205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

Commit message: modificaciones del PCB
Parts:
- renumbered J3 to J2, J2 to J3
Other:
- title: Puente_H_Fuente_AT -> Puente_H_Fuente_AT_SCH
- moved on the sheet: J3
