File: Tesis MIB/TESIS - Desarrollo/PCB/Bloque de control y FI/v2/Bloque de control y FI v2/Bloque de control y FI v2.kicad_pcb (KiCad board)
At the start: 2 copper layers, 95 x 80 mm, 37 parts, among them J1 AudioJack2, J2 Screw_Terminal_01x02, J3 Screw_Terminal_01x02, J4 Screw_Terminal_01x04, J5 FSR_b, J6 FSR_a, Q1 BF420, Q2 BF421, Q3 BF421, Q4 BF420, Q5 BF421, Q6 BF420, SW1 Decr, SW2 Inc, SW3 Acept, U1 LCD-016N002L, U2 PSoC4_kit049_(CY8C4245AXI-483), U3 TL082

Commit message: ultima
Parts:
- removed D1, D2: 1N4148, Diode_THT:D_DO-41_SOD81_P7.62mm_Horizontal
- removed the J4 at (47.8, 107.4)
- removed the Q3 at (58.4, 58.7)
- removed REF1, REF2, REF3: MountingHole_3.7mm, MountingHole:MountingHole_3.7mm
- removed RV4: 10k, Potentiometer_THT:Potentiometer_Bourns_3296W_Vertical
- removed SW1: Decr, Button_Switch_THT:SW_PUSH_6mm_H7.3mm
- removed SW2: Inc, Button_Switch_THT:SW_PUSH_6mm_H7.3mm
- removed SW3: Acept, Button_Switch_THT:SW_PUSH_6mm_H7.3mm
- added C1: 10uF, Capacitor_THT:CP_Radial_D5.0mm_P2.50mm, F.Cu at (123.6, 94.0)
- added C2: 33uF, Capacitor_THT:CP_Radial_D5.0mm_P2.50mm, F.Cu at (142.6, 95.5)
- added C3: 330nF, Capacitor_THT:C_Disc_D5.0mm_W2.5mm_P5.00mm, F.Cu at (140.8, 108.7)
- added C4: 330nF, Capacitor_THT:C_Disc_D5.0mm_W2.5mm_P5.00mm, F.Cu at (136.5, 108.7)
- added C5: 10nF, Capacitor_THT:C_Disc_D5.0mm_W2.5mm_P5.00mm, F.Cu at (148.9, 103.8)
- added C6: 10nF, Capacitor_THT:C_Disc_D5.0mm_W2.5mm_P5.00mm, F.Cu at (135.8, 100.7)
- added J10: Screw_Terminal_01x02, TerminalBlock:TerminalBlock_bornier-2_P5.08mm, F.Cu at (115.8, 113.4)
- added J11: 12%, Connector_Pin:Pin_D0.9mm_L10.0mm_W2.4mm_FlatFork, F.Cu at (152.7, 62.5)
- added J12: 8%, Connector_Pin:Pin_D0.9mm_L10.0mm_W2.4mm_FlatFork, F.Cu at (152.7, 65.5)
- added J13: 12%, Connector_Pin:Pin_D0.9mm_L10.0mm_W2.4mm_FlatFork, F.Cu at (149.1, 62.5)
- added J14: 16%, Connector_Pin:Pin_D0.9mm_L10.0mm_W2.4mm_FlatFork, F.Cu at (149.1, 59.4)
- added J15: GND_But, Connector_Pin:Pin_D0.9mm_L10.0mm_W2.4mm_FlatFork, F.Cu at (161.2, 110.0)
- added J16: Acept, Connector_Pin:Pin_D0.9mm_L10.0mm_W2.4mm_FlatFork, F.Cu at (168.3, 110.0)
- added J17: Inc, Connector_Pin:Pin_D0.9mm_L10.0mm_W2.4mm_FlatFork, F.Cu at (164.7, 110.0)
- added J2: Osc, Connector_Pin:Pin_D0.9mm_L10.0mm_W2.4mm_FlatFork, F.Cu at (152.1, 42.5)
- added J5: 16%, Connector_Pin:Pin_D0.9mm_L10.0mm_W2.4mm_FlatFork, F.Cu at (152.7, 59.4)
- added J6: 8%, Connector_Pin:Pin_D0.9mm_L10.0mm_W2.4mm_FlatFork, F.Cu at (149.1, 65.5)
- added J7: Decr, Connector_Pin:Pin_D0.9mm_L10.0mm_W2.4mm_FlatFork, F.Cu at (172.0, 110.0)
- added Q1: MPSA94, Proyecto_MIB:BF42X, F.Cu at (131.0, 63.2)
- added Q7: 13001, Proyecto_MIB:BF42X, F.Cu at (129.5, 49.4)
- added Q8: 13001, Proyecto_MIB:BF42X, F.Cu at (141.6, 49.6)
- added R1: 1k, Resistor_THT:R_Axial_DIN0207_L6.3mm_D2.5mm_P10.16mm_Horizontal, F.Cu at (156.1, 52.8)
- added R12: 680, Resistor_THT:R_Axial_DIN0207_L6.3mm_D2.5mm_P10.16mm_Horizontal, F.Cu at (121.7, 40.6)
- added R13: 680, Resistor_THT:R_Axial_DIN0207_L6.3mm_D2.5mm_P10.16mm_Horizontal, F.Cu at (127.3, 40.6)
- added R2: 390, Resistor_THT:R_Axial_DIN0207_L6.3mm_D2.5mm_P10.16mm_Horizontal, F.Cu at (124.6, 69.1)
- added R3: 390, Resistor_THT:R_Axial_DIN0207_L6.3mm_D2.5mm_P10.16mm_Horizontal, F.Cu at (124.6, 73.4)
- added R5: 10k, Resistor_THT:R_Axial_DIN0207_L6.3mm_D2.5mm_P10.16mm_Horizontal, F.Cu at (170.4, 60.3)
- added R9: 27k, Resistor_THT:R_Axial_DIN0207_L6.3mm_D2.5mm_P10.16mm_Horizontal, F.Cu at (163.1, 60.3)
- added REF**: MountingHole_3.2mm_M3, MountingHole:MountingHole_3.2mm_M3, F.Cu at (115.4, 58.8)
- added REF**: MountingHole_3.2mm_M3, MountingHole:MountingHole_3.2mm_M3, F.Cu at (115.7, 99.4)
- added REF**: MountingHole_3.2mm_M3, MountingHole:MountingHole_3.2mm_M3, F.Cu at (170.3, 79.9)
- added REF**: MountingHole_3.2mm_M3, MountingHole:MountingHole_3.2mm_M3, F.Cu at (214.5, 110.0)
- added REF**: MountingHole_3.2mm_M3, MountingHole:MountingHole_3.2mm_M3, F.Cu at (216.0, 41.5)
- added U4: ICL7660, Package_DIP:DIP-8_W7.62mm, F.Cu at (128.8, 88.0)
- added U5: L78L09_TO92, Package_TO_SOT_THT:TO-92_Inline_Wide, F.Cu at (131.0, 100.6)
- added U6: LM78L05_TO92, Package_TO_SOT_THT:TO-92_Inline_Wide, F.Cu at (149.0, 108.1)
- Q2: value BF421 -> MPSA94
- Q4: value BF420 -> MPSA94
- Q5: value BF421 -> 13001
- Q6: value BF420 -> 13001
- R11: renamed from R10; value 2k -> 2k2
- R4: renamed from R8; value 47k -> 33k
- R7: renamed from R9; value 10k -> 15k
- R8: renamed from R4; value 10k -> 12k
- RV1: renamed from RV3; value 50k -> 10k; footprint Potentiometer_THT:Potentiometer_Bourns_3296W_Vertical -> Potentiometer_THT:Potentiometer_ACP_CA9-V10_Vertical
- RV2: value 2k -> 5k
- U1: renamed from U3; footprint Package_DIP:DIP-8_W10.16mm_LongPads -> Package_DIP:DIP-8_W7.62mm
- moved R7 116.0 mm to (166.8, 60.3), turned to -90 degrees
- moved R10 102.1 mm to (156.0, 95.2), turned to 180 degrees
- moved R11 96.4 mm to (159.4, 60.3), turned to -90 degrees
- moved R6 94.9 mm to (162.2, 98.6)
- moved U1 93.6 mm to (163.4, 81.7)
- moved R4 93.6 mm to (152.0, 92.3)
- moved RV1 89.9 mm to (142.3, 70.9), turned to -90 degrees
- moved U2 81.0 mm to (197.9, 105.4)
- moved J1 81.0 mm to (161.5, 48.1)
- moved R14 81.0 mm to (193.9, 73.4)
- moved R15 81.0 mm to (196.9, 75.2)
- moved R16 81.0 mm to (183.7, 77.2)
- moved R17 81.0 mm to (183.7, 81.0)
- moved RV2 81.0 mm to (154.2, 106.9)
- moved RV3 81.0 mm to (204.8, 112.3)
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- renumbered J2 to J3, J3 to J4, J5 to J8, J6 to J9, Q1 to Q3, R7 to R10, R2 to R14, R1 to R15, R3 to R16, R5 to R17, RV1 to RV3, U1 to U3
Connections:
- J1 pad S: GND -> Net-(J2-Pin_1)
- Q2 pad 1: Net-(D1-K) -> Net-(Q2-E)
- Q2 pad 2: Net-(Q2-C) -> Net-(Q1-B)
- Q2 pad 3: Net-(Q1-B) -> /Control_y_salida/Iout
- Q3 pad 1: Net-(D1-K) -> Net-(Q3-E)
- Q3 pad 2: Net-(Q1-C) -> Net-(Q1-B)
- Q3 pad 3: Net-(Q1-B) -> Net-(Q3-B)
- Q4 pad 1: VEE -> Net-(Q4-E)
- Q4 pad 2: Net-(Q2-C) -> Net-(Q3-B)
- Q4 pad 3: Net-(Q2-C) -> Net-(Q4-C)
- Q5 pad 1: VCC -> Net-(Q5-E)
- Q5 pad 2: /Control_y_salida/Iout -> Net-(Q4-C)
- Q5 pad 3: Net-(Q1-C) -> Net-(Q4-C)
- Q6 pad 1: VEE -> Net-(Q6-E)
- Q6 pad 3: Net-(Q2-C) -> Net-(Q4-C)
- R11 pad 1: Net-(R10-Pad1) -> GND
- R11 pad 2: Net-(D1-A) -> Net-(Q4-E)
- R7 pad 1: Net-(R9-Pad1) -> GND
- RV1 pad 1: Net-(R9-Pad1) -> Net-(Q3-E)
- RV1 pad 2: Net-(R9-Pad1) -> Net-(Q3-E)
- RV1 pad 3: GND -> Net-(J13-Pin_1)
- U1 pad 1: Net-(Q1-B) -> Net-(Q3-B)
- U1 pad 2: Net-(D1-K) -> Net-(Q3-B)
- U1 pad 4: -12V -> -9V
- U1 pad 8: +12V -> +9V
Routing:
- net GND: track 230.7 -> 424.1 mm, vias 4 -> 5
- net Net-(Q4-C): track 0.00 -> 60.3 mm
- net +9V: track 0.00 -> 58.2 mm, vias 0 -> 2
- net -12V: track 52.8 -> 0.00 mm, vias 2 -> 0
- net Net-(Q3-B): track 0.00 -> 50.0 mm
- net +12V: track 33.2 -> 0.00 mm
- net Net-(Q4-E): track 0.00 -> 31.8 mm
- net Net-(D1-K): track 31.8 -> 0.00 mm
- net /Control_y_salida/+12V: track 0.00 -> 31.3 mm
- net -9V: track 0.00 -> 28.6 mm
- net Net-(Q2-C): track 25.1 -> 0.00 mm
- net Net-(J5-Pin_1): track 0.00 -> 23.8 mm
- net Net-(Q1-C): track 23.4 -> 0.00 mm
- net /Control_y_salida/IDAC_Pos: track 52.9 -> 31.8 mm
- net +5V: track 203.3 -> 182.2 mm, vias 6 -> 3
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- added copper zone on F.Cu, net GND
- added copper zone on B.Cu, net VCC
- added copper zone on B.Cu, net VEE
- removed copper zone on F.Cu, net +5V
Other:
- board size 95 x 80 mm -> 109.9 x 80 mm
- board text removed: "Electroestimulador por Corriente Tesis - MIB, FI-UNER García Cabrera, Jeremías A. Rev. 2.0 - 11/2023"
