File: Tesis MIB/TESIS - Desarrollo/PCB/Bloque de control y FI/v2/Bloque de control y FI v2/Bloque de control y FI v2.kicad_sch (KiCad schematic)
At the start: 3 parts, among them J1 AudioJack2, J8 Osc

Commit message: ultima
Parts:
- renumbered J8 to J2, R18 to R1
Other:
- sheet Control_y_salida ports: added none; removed +5V
- sheet Fuente ports: added none; removed +5V
Changed lines of the file:
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@@
-	(wire
-		(pts
-			(xy 156.21 87.63) (xy 170.18 87.63)
-		)
-		(stroke
-			(width 0)
-			(type default)
-		)
-	)
 	(wire
 		(pts
@@
 		(on_board yes)
 		(dnp no)
-		(property "Reference" "R18"
+		(property "Reference" "R1"
 			(at 217.932 93.472 0)
 			(effects
@@
 			(project "Bloque de control y FI v2"
 				(path "/d8b362ed-b66b-443a-9ff8-8e45e9f3933f"
-					(reference "R18")
+					(reference "R1")
 					(unit 1)
 				)
@@
 		(on_board yes)
 		(dnp no)
-		(property "Reference" "J8"
+		(property "Reference" "J2"
 			(at 219.71 90.17 0)
 			(effects
@@
 			(project "Bloque de control y FI v2"
 				(path "/d8b362ed-b66b-443a-9ff8-8e45e9f3933f"
-					(reference "J8")
+					(reference "J2")
 					(unit 1)
 				)
@@
 			)
 		)
-		(pin "+5V" input
-			(at 170.18 87.63 180)
-			(effects
-				(font
-					(size 1.27 1.27)
-				)
-				(justify left)
-			)
-		)
 		(pin "Iout" bidirectional
 			(at 208.28 81.28 0)
@@
 			)
 		)
-		(pin "+5V" input
-			(at 156.21 87.63 0)
-			(effects
-				(font
-					(size 1.27 1.27)
-				)
-				(justify right)
-			)
-		)
