File: Tesis MIB/TESIS - Desarrollo/PCB/Bloque de control y FI/v2/Bloque de control y FI v2/Control_y_salida.kicad_sch (KiCad schematic)
At the start: 40 parts, among them J10 1_8% - 2_12% - 3_16%, J5 FSR_b, J6 FSR_a, J7 1_8% - 2_12% - 3_16%, Q10 MPSA94, Q3 BF420, Q4 MPSA94, Q5 13001, Q6 13001, Q7 13001, Q8 13001, Q9 MPSA94, SW1 Decr, SW2 Inc, SW3 Acept, U1 TL082, U2 PSoC4_kit049_(CY8C4245AXI-483), U3 LCD-016N002L, U4 LT1054

Commit message: CAP 3 finalizado e inicio del 4to
Redactado la discución de resultados
Parts:
- J10, J7: footprint (none) -> Connector_PinHeader_1.00mm:PinHeader_1x03_P1.00mm_Vertical
Changed lines of the file:
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@@
 			)
 		)
-		(property "Footprint" ""
+		(property "Footprint" "Connector_PinHeader_1.00mm:PinHeader_1x03_P1.00mm_Vertical"
 			(at 196.85 80.01 0)
 			(effects
@@
 			)
 		)
-		(property "Footprint" ""
+		(property "Footprint" "Connector_PinHeader_1.00mm:PinHeader_1x03_P1.00mm_Vertical"
 			(at 195.58 80.01 0)
 			(effects

Commit message: ultima
Parts:
- removed C1, C2: 100uF x 16V, Capacitor_THT:CP_Radial_D6.3mm_P2.50mm, symbol Device:C_Polarized
- removed J10, J7: 1_8% - 2_12% - 3_16%, Connector_PinHeader_1.00mm:PinHeader_1x03_P1.00mm_Vertical, symbol Connector:Conn_01x03_Pin
- removed SW1: Decr, Button_Switch_THT:SW_PUSH_6mm_H7.3mm, symbol Switch:SW_Push
- removed SW2: Inc, Button_Switch_THT:SW_PUSH_6mm_H7.3mm, symbol Switch:SW_Push
- removed SW3: Acept, Button_Switch_THT:SW_PUSH_6mm_H7.3mm, symbol Switch:SW_Push
- removed U4: LT1054, Package_DIP:DIP-8_W7.62mm_LongPads, symbol Regulator_SwitchedCapacitor:LT1054
- added C1: 10uF, Capacitor_THT:CP_Radial_D5.0mm_P2.50mm, symbol Device:C_Polarized_Small
- added C2: 33uF, Capacitor_THT:CP_Radial_D5.0mm_P2.50mm, symbol Device:C_Polarized_Small
- added C3, C4: 330nF, Capacitor_THT:C_Disc_D5.0mm_W2.5mm_P5.00mm, symbol Device:C
- added C5, C6: 10nF, Capacitor_THT:C_Disc_D5.0mm_W2.5mm_P5.00mm, symbol Device:C
- added J11, J13: 12%, Connector_Pin:Pin_D0.9mm_L10.0mm_W2.4mm_FlatFork, symbol Connector:Conn_01x01_Male
- added J12, J6: 8%, Connector_Pin:Pin_D0.9mm_L10.0mm_W2.4mm_FlatFork, symbol Connector:Conn_01x01_Male
- added J14, J5: 16%, Connector_Pin:Pin_D0.9mm_L10.0mm_W2.4mm_FlatFork, symbol Connector:Conn_01x01_Male
- added J15: GND_But, Connector_Pin:Pin_D0.9mm_L10.0mm_W2.4mm_FlatFork, symbol Connector:Conn_01x01_Male
- added J16: Acept, Connector_Pin:Pin_D0.9mm_L10.0mm_W2.4mm_FlatFork, symbol Connector:Conn_01x01_Male
- added J17: Inc, Connector_Pin:Pin_D0.9mm_L10.0mm_W2.4mm_FlatFork, symbol Connector:Conn_01x01_Male
- added J7: Decr, Connector_Pin:Pin_D0.9mm_L10.0mm_W2.4mm_FlatFork, symbol Connector:Conn_01x01_Male
- added U4: ICL7660, Package_DIP:DIP-8_W7.62mm, symbol Regulator_SwitchedCapacitor:ICL7660
- added U5: L78L09_TO92, Package_TO_SOT_THT:TO-92_Inline_Wide, symbol Regulator_Linear:L78L09_TO92
- added U6: LM78L05_TO92, Package_TO_SOT_THT:TO-92_Inline_Wide, symbol Regulator_Linear:LM78L05_TO92
- Q1: renamed from Q10; footprint Package_TO_SOT_THT:TO-92_Inline -> Proyecto_MIB:BF42X
- Q2: renamed from Q9; footprint Package_TO_SOT_THT:TO-92_Inline -> Proyecto_MIB:BF42X
- Q4, Q5, Q6, Q7, Q8: footprint Package_TO_SOT_THT:TO-92_Inline -> Proyecto_MIB:BF42X
- R11: renamed from R7; value 3k3 -> 2k2
- R4: renamed from R3; value 47k -> 33k
- R5: renamed from R15; value 15k -> 10k
- R7: renamed from R5; value 24k -> 15k
- R8: renamed from R6; value 10k -> 12k
- R9: renamed from R17; value 33k -> 27k
- RV1: footprint Potentiometer_THT:Potentiometer_Bourns_3296W_Vertical -> Potentiometer_THT:Potentiometer_ACP_CA9-V10_Vertical
- RV2: renamed from RV3; value 2k -> 5k
- U1: footprint Package_DIP:DIP-8_W10.16mm_LongPads -> Package_DIP:DIP-8_W7.62mm
- renumbered J5 to J8, J6 to J9, R8 to R10, R9 to R12, R10 to R13, R11 to R14, R12 to R15, R13 to R16, R14 to R17, R1 to R2, R2 to R3, R4 to R6, RV4 to RV3
Connections:
- net +12V: now also C3.1, C4.1, U5.3 (VI), U6.3 (VI); no longer U1.8 (V+)
- net +5V: now also C5.1, U6.1 (VO)
- net But_Acept: now also J16.1 (Pin_1)
- net But_Dec: now also J7.1 (Pin_1)
- net But_Inc: now also J17.1 (Pin_1)
- net GND: now also C2.1, C3.2, C4.2, C5.2, C6.2, J15.1 (Pin_1), U4.3 (GND), U5.2 (GND), U6.2 (GND)
- net at R5.2: now also J5.1 (Pin_1)
- net at RV1.3: now also J13.1 (Pin_1), J14.1 (Pin_1), J6.1 (Pin_1)
- net at R7.2: now also J11.1 (Pin_1)
- net at R9.2: now also J12.1 (Pin_1)
- net -12V renamed -9V
- net -9V: now also C2.2, U4.5 (VOUT)
- new net: C1.1, U4.2 (CAP+)
- new net: C1.2, U4.4 (CAP-)
- new net +9V: C6.1, U1.8 (V+), U4.8 (V+), U5.1 (VO)
- no-connect marks 34 -> 33
