File: Tesis MIB/TESIS - Desarrollo/PCB/Bloque de control y FI/v2/Bloque de control y FI v2/Fuente.kicad_sch (KiCad schematic)
At the start: 3 parts, among them J2 Screw_Terminal_01x02, J3 Screw_Terminal_01x02, J9 Screw_Terminal_01x03

Commit message: ultima
Parts:
- removed J9: Screw_Terminal_01x03, symbol Connector:Screw_Terminal_01x03
- added J10: Screw_Terminal_01x02, TerminalBlock:TerminalBlock_bornier-2_P5.08mm, symbol Connector:Screw_Terminal_01x02
- renumbered J2 to J3, J3 to J4
Connections:
- net +12V: now also J10.2 (Pin_2)
- net GND: now also J10.1 (Pin_1)
